File: 5_volt_regulated/10V regulated power supply shematic.kicad_sch (KiCad schematic)
At the start: 12 parts, among them J2 (+10v, gnd), U1 LM317_TO-220

Commit message: nessesary commits inc changing the file name to harass paul
Parts:
- removed V1: VSIN, symbol Simulation_SPICE:VSIN
- added D5: LED, symbol Device:LED
- added F1: Fuse, symbol Device:Fuse
- added J1: Screw_Terminal_01x02, symbol Connector:Screw_Terminal_01x02
- added T1: 230V → 12V AC, 150mA, symbol Device:Transformer_1P_1S
Connections:
- net GND: now also D5.1 (K)
- net at R1.2: now also D5.2 (A)
- net at D1.1 (K), D2.2 (A): now also T1.4 (SB)
- net at D3.2 (A), D4.1 (K): now also T1.3 (SA)
- new net: F1.2, T1.1 (AA)
